File: mic5332/mic5332.kicad_pcb (KiCad board)
At the start: 2 copper layers, 30 x 25 mm, 24 parts, among them U1 MIC5332

Commit message: 6월9일
Parts:
- added G***: LOGO, mic5332:THEpeach, F.Cu at (135.3, 84.3)
- added H1: MountingHole_Pad, MountingHole:MountingHole_3.2mm_M3_Pad_Via, F.Cu at (114.7, 84.5)
- DIS1: renamed from disable2; footprint TestPoint:TestPoint_2Pads_Pitch2.54mm_Drill0.8mm -> Jumper:SolderJumper-2_P1.3mm_Open_TrianglePad1.0x1.5mm
- DIS2: renamed from disable1; footprint TestPoint:TestPoint_2Pads_Pitch2.54mm_Drill0.8mm -> Jumper:SolderJumper-2_P1.3mm_Open_TrianglePad1.0x1.5mm
- moved DIS2 1.78 mm to (129.4, 84.3)
- moved DIS1 1.67 mm to (122.8, 84.3)
- renumbered V_IN to 5V_IN
Routing:
- net Net-(EN2-Pad1): track 16.5 -> 12.2 mm, vias 1 -> 2
- net GND: vias 6 -> 3
Other:
- board text added: "2020.06.10"
- board text added: "3v3 REGUL"
- board text added: "Park Jung Eun"
- board text removed: "2020.05.28"
- board text removed: "PEACH"
- board text removed: "Park JungEun"
