File: mic5332/mic5332.sch (KiCad schematic (older format))
At the start: 24 parts, among them U1 MIC5332-SSYMT-TR

Commit message: 6월9일
Parts:
- added H1: MountingHole_Pad, MountingHole:MountingHole_3.2mm_M3_Pad_Via, symbol Mechanical:MountingHole_Pad
- JP1, JP2: footprint TestPoint:TestPoint_2Pads_Pitch2.54mm_Drill0.8mm -> Jumper:SolderJumper-2_P1.3mm_Open_TrianglePad1.0x1.5mm
Connections:
- net GND: now also H1.1
Changed lines of the file:
@@
 encoding utf-8
 Sheet 1 1
-Title ""
-Date ""
-Rev ""
-Comp ""
-Comment1 ""
+Title "MIC5332"
+Date "2020-06-09"
+Rev "LAST"
+Comp "THE PEACH"
+Comment1 "add Mounting Hole"
 Comment2 ""
 Comment3 ""
-Comment4 ""
+Comment4 "Author : Park Jung Eun"
 $EndDescr
 Wire Wire Line
@@
 F 0 "JP2" H 3550 3600 50  0000 C CNN
 F 1 "Jumper_2_Open" H 3550 3350 50  0000 C CNN
-F 2 "TestPoint:TestPoint_2Pads_Pitch2.54mm_Drill0.8mm" H 3550 3500 50  0001 C CNN
+F 2 "Jumper:SolderJumper-2_P1.3mm_Open_TrianglePad1.0x1.5mm" H 3550 3500 50  0001 C CNN
 F 3 "~" H 3550 3500 50  0001 C CNN
 	1    3550 3500
@@
 F 0 "JP1" H 3000 3600 50  0000 C CNN
 F 1 "Jumper_2_Open" H 2900 3350 50  0000 C CNN
-F 2 "TestPoint:TestPoint_2Pads_Pitch2.54mm_Drill0.8mm" H 3000 3500 50  0001 C CNN
+F 2 "Jumper:SolderJumper-2_P1.3mm_Open_TrianglePad1.0x1.5mm" H 3000 3500 50  0001 C CNN
 F 3 "~" H 3000 3500 50  0001 C CNN
 	1    3000 3500
@@
 Wire Wire Line
 	5700 3600 7800 3600
+$Comp
+L Mechanical:MountingHole_Pad H1
+U 1 1 5EDF7700
+P 2550 2550
+F 0 "H1" H 2650 2599 50  0000 L CNN
+F 1 "MountingHole_Pad" H 2650 2508 50  0000 L CNN
+F 2 "MountingHole:MountingHole_3.2mm_M3_Pad_Via" H 2550 2550 50  0001 C CNN
+F 3 "~" H 2550 2550 50  0001 C CNN
+	1    2550 2550
+	1    0    0    -1
+$EndComp
+Wire Wire Line
+	2550 2650 2550 2800
+$Comp
+L power:GND #PWR0101
+U 1 1 5EDF94BF
+P 2550 2800
+F 0 "#PWR0101" H 2550 2550 50  0001 C CNN
+F 1 "GND" H 2555 2627 50  0000 C CNN
+F 2 "" H 2550 2800 50  0001 C CNN
+F 3 "" H 2550 2800 50  0001 C CNN
+	1    2550 2800
+	1    0    0    -1
+$EndComp
 $EndSCHEMATC
