File: sensors/sensors.sch (KiCad schematic (older format))
At the start: 22 parts, among them J1 Conn_01x16_Male, J2 Conn_01x16_Male, SW1 SW_DIP_x02, U1 IST8310, U2 MPU-9250, U3 MS5611-01BA, U4 ICM-20602

Commit message: 6월9일
Parts:
- removed J1, J2: Conn_01x16_Male, Connector_PinHeader_2.54mm:PinHeader_1x16_P2.54mm_Vertical, symbol Connector:Conn_01x16_Male
- removed SW1: SW_DIP_x02, Button_Switch_SMD:SW_DIP_SPSTx02_Slide_KingTek_DSHP02TJ_W5.25mm_P1.27mm_JPin, symbol Switch:SW_DIP_x02
- added C12, C13: 22uF, Capacitor_SMD:C_0805_2012Metric_Pad1.15x1.40mm_HandSolder, symbol Device:C
- added J1: Conn_01x14_Male, Connector_PinHeader_2.54mm:PinHeader_1x14_P2.54mm_Vertical, symbol Connector:Conn_01x14_Male
- added JP1, JP2: Jumper, Capacitor_SMD:C_0402_1005Metric, symbol Device:Jumper_NO_Small
- C1: value 10n/4V -> 10n; manf# (none) -> ‎C0402C103K4RECAUTO
- C2: value 0u1/4V -> 0u1; manf# (none) -> CL10A104KA8NNNC
- C6: value 0u1/2V -> 0u1
- U4: def# (none) -> https://www.digikey.kr/product-detail/ko/tdk-invensense/ICM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
- renumbered R3 to R1, R4 to R2, R1 to R3, R2 to R4
Connections:
- net GND: now also C12.1, C13.1, J1.2 (Pin_2), JP1.2, JP2.2
- net INT_20602: now also J1.10 (Pin_10)
- net INT_9250: now also J1.5 (Pin_5)
- net MISO: now also J1.8 (Pin_8)
- net MOSI: now also J1.7 (Pin_7)
- net READY: now also J1.12 (Pin_12)
- net RESET: now also J1.11 (Pin_11)
- net SCL: now also J1.14 (Pin_14)
- net SCLK: now also J1.6 (Pin_6)
- net SDA: now also J1.13 (Pin_13)
- net VDD: now also C12.2, C13.2, J1.1 (Pin_1)
- net ~CS_20602: now also J1.9 (Pin_9)
- net ~CS_5611: now also J1.3 (Pin_3)
- net ~CS_9250: now also J1.4 (Pin_4)
- net ADRESS0: no longer names the net of R3.1, U1.5 (CAD0)
- net ADRESS0: now also JP1.1
- net ADRESS1: no longer names the net of R4.1, U1.6 (CAD1)
- net ADRESS1: now also JP2.1
Other:
- moved on the sheet: C10, C11, C7, C8, C9, R3, R4, U3, U4
