File: omnibusFC/omnibusFC.sch (KiCad schematic (older format))
At the start: 98 parts, among them J1 Conn03, J10 5PIN_CON, J11 Conn03, J12 Con02, J13 5PIN_CON, J14 8PIN_CON, J15 USB_B_Micro, J16 8PIN_CON, J2 Conn03, J3 Con02, J4 6PIN_CON, J5 Con02, J6 Conn03, J7 Conn03, J8 Micro_SD_Card_Det, J9 8PIN_CON, Q1 MMBT3904, Q2 MMBT3904, Q3 MMBT3904, SW1 SW_Push, U1 STM32F405RGTx, U2 MIC5332-SSYMT-TR, U3 MS5611-01BA, U4 MPU-9250, U5 MP1593, U6 INA139, Y1 Crystal

Commit message: 6월16일
Parts:
- removed J10, J13: 5PIN_CON, symbol omnibusFC:5PIN_CON
- removed J14, J16, J9: 8PIN_CON, symbol omnibusFC:8PIN_CON
- removed J4: 6PIN_CON, symbol omnibusFC:6PIN_CON
- removed U1: STM32F405RGTx, Package_QFP:LQFP-64_10x10mm_P0.5mm, symbol MCU_ST_STM32F4:STM32F405RGTx
- removed U2: MIC5332-SSYMT-TR, TMLF-8_MCH, symbol mic5332:MIC5332-SSYMT-TR
- removed U4: MPU-9250, Sensor_Motion:InvenSense_QFN-24_3x3mm_P0.4mm, symbol Sensor_Motion:MPU-9250
- removed U5: MP1593, symbol omnibusFC:MP1593
- added C1, C10, C13, C2, C21, C4, C5, C6, C9: 0u1, Capacitor_SMD:C_0402_1005Metric, symbol Device:C
- added H1, H2, H3, H4: Hole_Pad, MountingHole:MountingHole_3mm_Pad, symbol Mechanical:MountingHole_Pad
- added J1, J8: Conn_03, Connector_JST:JST_GH_SM03B-GHS-TB_1x03-1MP_P1.25mm_Horizontal, symbol Connector_Generic_MountingPin:Conn_01x03_MountingPin
- added J10, J11, J4: Conn_06, Connector_JST:JST_GH_SM06B-GHS-TB_1x06-1MP_P1.25mm_Horizontal, symbol Connector_Generic_MountingPin:Conn_01x06_MountingPin
- added J5: Conn_04, Connector_JST:JST_GH_SM04B-GHS-TB_1x04-1MP_P1.25mm_Horizontal, symbol Connector_Generic_MountingPin:Conn_01x04_MountingPin
- added R18, R21: 1M, Resistor_SMD:R_0402_1005Metric, symbol Device:R
- added U1: STM32F405RGT6, Package_QFP:LQFP-64_10x10mm_P0.5mm, symbol omnibusFC:STM32F405RGT6
- added U2: MP1593, omnibusFC:mp1593, symbol omnibusFC:MP1593
- added U3: MPU-9250, omnibusFC:mpu9250, symbol omnibusFC:MPU-9250
- added U4: MIC5332-SSYMT-TR, omnibusFC:TMLF-8_MCH, symbol mic5332:MIC5332-SSYMT-TR
- C11: renamed from C1; footprint (none) -> Capacitor_SMD:C_0402_1005Metric
- C12: renamed from C2; footprint (none) -> Capacitor_SMD:C_0402_1005Metric
- C14: renamed from C9; footprint (none) -> Capacitor_SMD:C_0402_1005Metric
- C19: renamed from C8; footprint (none) -> Capacitor_SMD:C_0805_2012Metric
- C20: renamed from C3; footprint (none) -> Capacitor_SMD:C_0402_1005Metric
- C23: renamed from C11; footprint (none) -> Capacitor_SMD:C_0402_1005Metric
- C24: renamed from C18; footprint (none) -> Capacitor_SMD:C_0805_2012Metric
- C25: renamed from C19; footprint (none) -> Capacitor_SMD:C_0402_1005Metric
- C26: renamed from C20; footprint (none) -> Capacitor_SMD:C_0402_1005Metric
- C27: renamed from C13; footprint (none) -> Capacitor_SMD:C_0402_1005Metric
- C30: renamed from C4; footprint (none) -> Capacitor_SMD:C_0402_1005Metric
- C31: renamed from C10; footprint (none) -> Capacitor_SMD:C_0805_2012Metric_Pad1.15x1.40mm_HandSolder
- C46: renamed from C5; footprint (none) -> Capacitor_SMD:C_0402_1005Metric
- C47: renamed from C15; footprint (none) -> Capacitor_SMD:C_0805_2012Metric
- C48: renamed from C17; footprint (none) -> Capacitor_SMD:C_0402_1005Metric
- C49: renamed from C14; footprint (none) -> Capacitor_SMD:C_0402_1005Metric
- C50: renamed from C12; footprint (none) -> Capacitor_SMD:C_0402_1005Metric
- C51: renamed from C16; footprint (none) -> Capacitor_SMD:C_0805_2012Metric
- C7: footprint (none) -> Capacitor_SMD:C_0402_1005Metric
- C8: renamed from C6; footprint (none) -> Capacitor_SMD:C_0402_1005Metric
- D1: renamed from D3; footprint (none) -> Diode_SMD:D_SOD-323
- D2: footprint (none) -> Diode_SMD:D_SOD-323
- D3: renamed from D1; footprint (none) -> Diode_SMD:D_SOD-323
- D5: footprint (none) -> LED_SMD:LED_0603_1608Metric_Pad1.05x0.95mm_HandSolder
- D6: renamed from D4; footprint (none) -> LED_SMD:LED_0603_1608Metric_Pad1.05x0.95mm_HandSolder
- D8: renamed from D6; footprint (none) -> Diode_SMD:D_SMA
- J12: renamed from J7; footprint (none) -> Connector_PinSocket_2.54mm:PinSocket_1x03_P2.54mm_Vertical
- J13: renamed from J6; footprint (none) -> Connector_PinSocket_2.54mm:PinSocket_1x03_P2.54mm_Vertical
- J14: renamed from J1; footprint (none) -> Connector_PinSocket_2.54mm:PinSocket_1x03_P2.54mm_Vertical
- J15: renamed from J2; footprint (none) -> Connector_PinSocket_2.54mm:PinSocket_1x03_P2.54mm_Vertical
- J2: renamed from J12; footprint (none) -> Connector_PinSocket_2.54mm:PinSocket_1x02_P2.54mm_Vertical
- J6: renamed from J3; footprint (none) -> Connector_PinSocket_2.54mm:PinSocket_1x02_P2.54mm_Vertical
- J7: renamed from J11; footprint (none) -> Connector_PinSocket_2.54mm:PinSocket_1x03_P2.54mm_Vertical
- J9: renamed from J5; footprint (none) -> Connector_PinSocket_2.54mm:PinSocket_1x02_P2.54mm_Vertical
- L1: footprint (none) -> Inductor_SMD:L_6.3x6.3_H3
- R1: renamed from R23; value R -> 330; footprint (none) -> Resistor_SMD:R_0402_1005Metric
- R10: renamed from R18; footprint (none) -> Resistor_SMD:R_0402_1005Metric
- R11: renamed from R15; footprint (none) -> Resistor_SMD:R_0402_1005Metric
- R12: renamed from R17; footprint (none) -> Resistor_SMD:R_0402_1005Metric
- R13: renamed from R12; footprint (none) -> Resistor_SMD:R_0402_1005Metric
- R14: renamed from R9; footprint (none) -> Resistor_SMD:R_0402_1005Metric
- R15: renamed from R19; footprint (none) -> Resistor_SMD:R_0402_1005Metric
- R16: renamed from R13; footprint (none) -> Resistor_SMD:R_0402_1005Metric
- R17: renamed from R1; footprint (none) -> Resistor_SMD:R_0402_1005Metric
- R19: renamed from R7; footprint (none) -> Resistor_SMD:R_0402_1005Metric
- R2: renamed from R24; value R -> 330; footprint (none) -> Resistor_SMD:R_0402_1005Metric
- R20: renamed from R6; footprint (none) -> Resistor_SMD:R_0402_1005Metric
- R3: renamed from R16; value R -> 50k; footprint (none) -> Resistor_SMD:R_0402_1005Metric
- R31: renamed from R30; footprint (none) -> Resistor_SMD:R_0402_1005Metric
- R32: renamed from R28; footprint (none) -> Resistor_SMD:R_Shunt_Vishay_WSR2_WSR3
- R38: renamed from R26; footprint (none) -> Resistor_SMD:R_0402_1005Metric
- R39: renamed from R31; footprint (none) -> Resistor_SMD:R_0402_1005Metric
- R4: renamed from R14; value R -> 330; footprint (none) -> Resistor_SMD:R_0402_1005Metric
- R40: renamed from R29; footprint (none) -> Resistor_SMD:R_0402_1005Metric
- R41: renamed from R27; footprint (none) -> Resistor_SMD:R_0402_1005Metric
- R42: renamed from R32; footprint (none) -> Resistor_SMD:R_0402_1005Metric
- R47: renamed from R4; footprint (none) -> Resistor_SMD:R_0402_1005Metric
- R48: renamed from R3; footprint (none) -> Resistor_SMD:R_0402_1005Metric
- R49: renamed from R5; footprint (none) -> Resistor_SMD:R_0402_1005Metric
- R5: renamed from R11; value R -> 10k; footprint (none) -> Resistor_SMD:R_0402_1005Metric
- R50: renamed from R2; footprint (none) -> Resistor_SMD:R_0402_1005Metric
- R51: renamed from R8; footprint (none) -> Resistor_SMD:R_0402_1005Metric
- R52: renamed from R25; footprint (none) -> Resistor_SMD:R_0402_1005Metric
- R6: renamed from R21; footprint (none) -> Resistor_SMD:R_0402_1005Metric
- R7: renamed from R20; footprint (none) -> Resistor_SMD:R_0402_1005Metric
- R8: renamed from R10; footprint (none) -> Resistor_SMD:R_0402_1005Metric
- R9: renamed from R22; value R -> 10k; footprint (none) -> Resistor_SMD:R_0402_1005Metric
- SW1: footprint (none) -> Button_Switch_SMD:SW_SPST_B3U-1000P
- TP1: renamed from TP9; footprint (none) -> TestPoint:TestPoint_Pad_D1.0mm
- TP11: renamed from TP8; footprint (none) -> TestPoint:TestPoint_Pad_D1.0mm
- TP12: renamed from TP5; footprint (none) -> TestPoint:TestPoint_Pad_D1.0mm
- TP13: renamed from TP7; footprint (none) -> TestPoint:TestPoint_Pad_D1.0mm
- TP2: renamed from TP6; footprint (none) -> TestPoint:TestPoint_Pad_D1.0mm
- TP23: renamed from TP1; footprint (none) -> TestPoint:TestPoint_Pad_D1.0mm
- TP3: renamed from TP4; footprint (none) -> TestPoint:TestPoint_Pad_D1.0mm
- TP4: renamed from TP10; footprint (none) -> TestPoint:TestPoint_Pad_D1.0mm
- TP5: renamed from TP2; footprint (none) -> TestPoint:TestPoint_Pad_D1.0mm
- TP6: renamed from TP3; footprint (none) -> TestPoint:TestPoint_Pad_D1.0mm
- TP7: renamed from TP11; footprint (none) -> TestPoint:TestPoint_Pad_D1.0mm
- TP8: renamed from TP12; footprint (none) -> TestPoint:TestPoint_Pad_D1.0mm
- U10: renamed from J8; footprint (none) -> Connector_Card:microSD_HC_Molex_104031-0811
- U9: renamed from U3; footprint Package_LGA:LGA-8_3x5mm_P1.25mm -> omnibusFC:ms5611
- USB1: renamed from J15; footprint (none) -> Connector_USB:USB_Micro-B_Molex_47346-0001
- Y1: footprint (none) -> Crystal:Crystal_SMD_MicroCrystal_CC7V-T1A-2Pin_3.2x1.5mm
- renumbered Q2 to Q1, Q3 to Q2, Q1 to Q3, U6 to U11
Connections:
- net BOOT0: now also U1.60 (BOOT0)
- net BUZZER: now also U1.56 (PB4)
- net CRNT: now also U1.9 (PC1)
- net ESC_5V: now also J11.2 (Pin_2)
- net GND: now also C1.1, C10.2, C13.2, C2.2, C21.2, C4.2, C5.2, C6.2, C9.2, H1.1, H2.1, H3.1, H4.1, J1.1 (Pin_1), J1.MP (MountPin), J10.4 (Pin_4), J10.MP (MountPin), J11.1 (Pin_1), J11.MP (MountPin), J4.1 (Pin_1), J4.MP (MountPin), J5.1 (Pin_1), J5.MP (MountPin), J8.2 (Pin_2), J8.MP (MountPin), R18.2, R21.1, U1.12 (VSSA), U1.18 (VSS), U1.28 (PB2), U1.63 (VSS), U2.4 (GND), U2.9 (EP), U3.11 (FSYNC), U3.18 (GND), U3.20 (RESV_GND), U4.2 (GND), U4.9; no longer U10.11 (SHIELD), USB1.6 (Shield)
- net INT_9250: now also U1.24 (PC4), U3.12 (INT)
- net LED_STRIP: now also J1.3 (Pin_3), U1.54 (PD2)
- net RC_CH1: now also U1.61 (PB8)
- net RC_CH3: now also J10.5 (Pin_5), U1.37 (PC6)
- net RC_CH4: now also J10.6 (Pin_6), U1.38 (PC7)
- net SD_DET: now also U1.59 (PB7)
- net SPI1_MISO: now also U1.22 (PA6), U3.9 (AD0/MISO)
- net SPI1_MOSI: now also U1.23 (PA7), U3.24 (SDA/MOSI)
- net SPI1_SCLK: now also U1.21 (PA5), U3.23 (SCL/SCLK)
- net SPI2_MISO: now also U1.35 (SPI2_MISO)
- net SPI2_MOSI: now also U1.36 (SIP2_MOSI)
- net SPI2_SCLK: now also U1.34 (SPI2_CLK)
- net SPI3_MISO: now also J4.5 (Pin_5), U1.52 (SPI3_MISO)
- net SPI3_MOSI: now also J4.3 (Pin_3), U1.53 (SPI3_MOSI)
- net SPI3_SCL: now also J4.4 (Pin_4), U1.51 (SPI3_CLK)
- net STAT: now also U1.57 (PB5)
- net Servo_out1: now also J11.6 (Pin_6), U1.26 (PB0)
- net Servo_out2: now also J11.5 (Pin_5), U1.27 (PB1)
- net Servo_out3: now also J11.3 (Pin_3), U1.17 (PA3)
- net Servo_out4: now also J11.4 (Pin_4), U1.16 (PA2)
- net Servo_out5: now also U1.15 (PA1)
- net Servo_out6: now also U1.41 (PA8)
- net UART3_RX: now also J10.1 (Pin_1), U1.30 (I2C_SDA/UART3_RX)
- net UART3_TX: now also J10.2 (Pin_2), U1.29 (I2C_SDA/UART3_TX)
- net USART_RX: now also Q1.3 (C), R5.1, J5.4 (Pin_4), J8.3 (Pin_3), U1.43 (UART1_RX); no longer C14.1, C20.1, C30.1, C31.1, C46.1, D5.2 (A), R1.1, R17.2, R47.2, R48.2, R49.2, R5.2, R50.2, R51.2, R8.2, SW1.2, TP7.1, U10.4 (VDD), U9.1 (VDD)
- net USART_TX: now also J5.3 (Pin_3), U1.42 (UART1_TX)
- net USB_DN: now also U1.44 (OTG_FS_DM)
- net USB_DP: now also U1.45 (OTG_FS_DP)
- net VBAT_ADC: now also U1.10 (PC2)
- net VBUS_SEN: now also U1.25 (PC5)
- net VCC5: now also J1.2 (Pin_2), J10.3 (Pin_3), J5.2 (Pin_2), U4.1 (VIN)
- net VCC_RC: now also J4.2 (Pin_2), U4.8 (VOUT1)
- net ~EX_SPI3_CS: now also J4.6 (Pin_6), U1.58 (PB6)
- net ~SPI1_SS: now also U1.20 (PA4), U3.22 (~CS)
- net ~SPI2_SS: now also U1.33 (~SPI2_SS)
- net ~SPI3_SS: now also U1.50 (~SPI3_SS)
- net at C24.1, R32.1, R41.2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: now also U2.2 (IN)
- net at R8.1: now also U1.11 (PC3)
- net at TP23.1: now also U1.14 (PA0)
- net at C11.1: now also U1.31 (VCAP_1)
- net at TP12.1: now also U1.39 (PC8)
- net at TP13.1: now also U1.40 (PC9)
- net at TP5.1: now also U1.46 (JTAG_SWDIO)
- net at C12.1: now also U1.47 (VCAP_2)
- net at TP6.1: now also U1.49 (JTAG_SWCLK)
- net at Y1.1: now also U1.5 (PH0)
- net at Y1.2: now also U1.6 (PH1)
- net at TP11.1: now also U1.62 (PB9)
- net at R17.1: now also U1.7 (NRST)
- net at C23.1: now also U3.10 (REGOUT)
- net at R15.2: now also U4.4 (EN2)
- net at R10.2: now also U4.5 (EN1)
- net at C8.1: now also U4.6 (CSET2)
- net at R41.1: now also U2.7 (EN)
- net at C25.1: now also U2.8 (SS)
- net at C26.1, C49.2: now also U2.6 (COMP)
- net at R39.1, R40.2: now also U2.5 (FB)
- net at C50.1, D8.1 (K), L1.1: now also U2.3 (SW)
- net at C50.2: now also U2.1 (BS)
- new net: C1.2, R18.1, U10.11 (SHIELD)
- new net: C2.1, R21.2, USB1.6 (Shield)
- new net VCC3v3: C10.1, C13.1, C14.1, C20.1, C21.1, C30.1, C31.1, C4.1, C46.1, C5.1, C6.1, C9.1, D5.2 (A), J8.1 (Pin_1), R1.1, R17.2, R47.2, R48.2, R49.2, R5.2, R50.2, R51.2, R8.2, SW1.2, TP7.1, U1.1 (VBAT), U1.13 (VDDA), U1.19 (VDD), U1.32 (VDD), U1.48 (VDD), U1.64 (VDD), U10.4 (VDD), U3.1 (RESV_VDDIO), U3.13 (VDD), U3.8 (VDDIO), U4.7 (VOUT2), U9.1 (VDD)
- no-connect marks 12 -> 7
Other:
- moved on the sheet: C11, C12, R17, R47, R48, R49, R5, R50, R51, R8, TP11, TP12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
